File: swich-payload.kicad_pcb (KiCad board)
At the start: 2 copper layers, 0 parts

Commit message: final
Parts:
- added BT1: Battery_Cell, EasyEDA:BAT-SMD_BHSD-2032-SM, B.Cu at (78.0, 95.5)
- added C1: 0.1 uF, Capacitor_SMD:C_0805_2012Metric, F.Cu at (71.0, 102.0)
- added C2: 10 uF, Capacitor_SMD:C_0805_2012Metric, F.Cu at (71.0, 100.0)
- added JP1: SolderJumper_2_Open, Jumper:SolderJumper-2_P1.3mm_Open_Pad1.0x1.5mm, F.Cu at (74.2, 100.7)
- added P1: USB_C_Plug_USB2.0, EasyEDA:USB-C-SMD_TYPE-C-31-G-10, F.Cu at (77.8, 109.0)
- added SW2: SW_Push, EasyEDA:SW-SMD_L3.0-W2.5-P3.40-LS4.0-EH, F.Cu at (73.3, 104.8)
- added SW3: TS6635PA 250GF TACTILE SWITCH, EasyEDA:SW-SMD_4P-L6.4-W6.3-P4.00-LS9.5, F.Cu at (78.0, 94.8)
- added TP1: TestPoint_Square, TestPoint:TestPoint_Pad_D2.0mm, F.Cu at (68.5, 108.5)
- added TP2: TestPoint_Square, TestPoint:TestPoint_Pad_D2.0mm, F.Cu at (68.5, 105.0)
- added TP3: TestPoint_Square, TestPoint:TestPoint_Pad_D1.0mm, F.Cu at (75.0, 103.0)
- added TP5: TestPoint_Square, TestPoint:TestPoint_Pad_D1.0mm, F.Cu at (81.0, 104.0)
- added TP6: TestPoint_Square, TestPoint:TestPoint_Pad_D2.0mm, F.Cu at (87.5, 108.5)
- added TP7: TestPoint_Square, TestPoint:TestPoint_Pad_D2.0mm, F.Cu at (85.0, 110.5)
- added TP8: TestPoint_Square, TestPoint:TestPoint_Pad_D2.0mm, F.Cu at (87.5, 98.0)
- added U2: CH554P, Package_DFN_QFN:QFN-16-1EP_3x3mm_P0.5mm_EP1.9x1.9mm, F.Cu at (77.8, 102.0)
- added U3: GL-1615RGB01-B, EasyEDA:LED-SMD_4P-L1.6-W1.5-BL-C9900013097, F.Cu at (80.5, 99.8)
- added U4: ZD25WD20CTIGT, EasyEDA:SOP-8_L4.9-W3.9-P1.27-LS6.0-BL, F.Cu at (84.5, 102.1)
Routing:
- net VCC: track 0.00 -> 28.7 mm, vias 0 -> 1
- net /SCK: track 0.00 -> 20.0 mm, vias 0 -> 2
- net /SI: track 0.00 -> 17.8 mm, vias 0 -> 2
- net /USB CC: track 0.00 -> 16.5 mm, vias 0 -> 2
- net /SO: track 0.00 -> 15.8 mm, vias 0 -> 2
- net GND: track 0.00 -> 13.4 mm, vias 0 -> 10
- net /USB D-: track 0.00 -> 12.1 mm, vias 0 -> 2
- net /USB D+: track 0.00 -> 11.7 mm, vias 0 -> 2
- net /BUTTON: track 0.00 -> 9.44 mm, vias 0 -> 2
- net /RST: track 0.00 -> 6.89 mm
- net /RBG R: track 0.00 -> 5.43 mm
- net /CS: track 0.00 -> 4.95 mm
- net /RGB G: track 0.00 -> 2.60 mm
- net Net-(JP1-B): track 0.00 -> 2.35 mm
- net /RGB B: track 0.00 -> 1.67 mm
- added copper zone on B.Cu, net GND
Other:
- board outline added: 23 x 34 mm
- board text added: "GND"
- board text added: "Pever3ll"
- board text added: "SCK"
- board text added: "SI"
- board text added: "SO"
- board text added: "VCC"
